Commit message: simulation works

File: src/meca500_world/models/meca500/meca500.urdf (robot description, URDF)
Before this commit: robot meca_500_r3, 7 links, 6 joints
Links:
- link meca_axis_1_link: mass 1.0 -> 1.2
- link meca_axis_3_link: mass 1.0 -> 0.8
- link meca_axis_4_link: mass 1.0 -> 0.6
- link meca_axis_5_link: mass 1.0 -> 0.5
- link meca_axis_6_link: mass 1.0 -> 0.3
- link meca_base_link: mass 1.0 -> 3.0

Commit message: working rgbd camera

File: src/meca500_world/models/meca500/meca500.urdf (robot description, URDF)
Before this commit: robot meca_500_r3, 7 links, 6 joints
Links:
- added link camera_link, mass 0.1; collision box size=0.05 0.05 0.05; visual box size=0.05 0.05 0.05
Joints:
- added joint camera_joint: type fixed, parent meca_axis_6_link, child camera_link, origin xyz=0 0 0.1 rpy=0 0 0

Commit message: aggiunto modello kinect

File: src/meca500_world/models/meca500/meca500.urdf (robot description, URDF)
Before this commit: robot meca_500_r3, 8 links, 7 joints
Links:
- link camera_link: mass 0.1 -> 0.5; geometry collision mesh filename=../../meshes/kinect.dae; visual mesh filename=../../meshes/kinect.dae
