Commit message: supports dynamic camera refresh rate configuration

File: src/meca500_world/models/meca500/meca500.xacro (robot description, xacro)
@@ -1,8 +1,6 @@
 <?xml version="1.0" encoding="utf-8"?>
-<!-- =================================================================================== -->
-<!-- |    This document was autogenerated by xacro from meca_500_r3.urdf.xacro         | -->
-<!-- |    EDITING THIS FILE BY HAND IS NOT RECOMMENDED                                 | -->
-<!-- =================================================================================== -->
-<robot name="meca_500_r3">
+<robot xmlns:xacro="http://www.ros.org/wiki/xacro" name="firefighter">
+  <xacro:arg name="camera_update_rate" default="60"/>
+  <xacro:property name="camera_update_rate" value="$(arg camera_update_rate)"/>
   <!-- Base link is the center of the robot's bottom plate -->
   <link name="meca_base_link">
@@ -295,5 +293,5 @@
   <gazebo reference="camera_link">
   <sensor name="rgbd_camera" type="rgbd_camera">
-    <update_rate>30.0</update_rate>
+    <update_rate>${camera_update_rate}</update_rate>
     <topic>rgbd_camera</topic>
     <camera>

Commit message: added designed camera holder to project

File: src/meca500_world/models/meca500/meca500.xacro (robot description, xacro)
@@ -3,4 +3,428 @@
   <xacro:arg name="camera_update_rate" default="60"/>
   <xacro:property name="camera_update_rate" value="$(arg camera_update_rate)"/>
+  <xacro:macro name="sensor_d435i" params="parent
+                                          name:=camera
+                                          topics_ns:=camera
+                                          visualize:=false
+                                          align_depth:=false
+                                          enable_pointCloud:=false
+                                          unite_imu_method:=false
+                                          accel_fps:=250
+                                          gyro_fps:=400
+                                          clip_distance:=-1.0
+                                          depth_width:=1280
+                                          depth_height:=720
+                                          depth_fps:=30
+                                          infra_width:=640
+                                          infra_height:=480
+                                          infra_fps:=30
+                                          color_width:=1920
+                                          color_height:=1080
+                                          color_fps:=30
+                                          *origin">
+    <xacro:property name="M_PI" value="3.1415926535897931"/>
+    <!-- The following values are approximate, and the camera node
+     publishing TF values with actual calibrated camera extrinsic values -->
+    <xacro:property name="d435i_cam_depth_to_left_ir_offset" value="0.0"/>
+    <xacro:property name="d435i_cam_depth_to_right_ir_offset" value="-0.050"/>
+    <xacro:property name="d435i_cam_depth_to_color_offset" value="0.015"/>
+    <!-- The following values model the aluminum peripherial case for the
+  	D435 camera, with the camera joint represented by the actual
+  	peripherial camera tripod mount -->
+    <xacro:property name="d435i_cam_width" value="0.090"/>
+    <xacro:property name="d435i_cam_height" value="0.025"/>
+    <xacro:property name="d435i_cam_depth" value="0.02505"/>
+    <xacro:property name="d435i_cam_mount_from_center_offset" value="0.0149"/>
+    <!-- The following offset is relative the the physical D435 camera peripherial
+  	camera tripod mount -->
+    <xacro:property name="d435i_cam_depth_px" value="${d435i_cam_mount_from_center_offset}"/>
+    <xacro:property name="d435i_cam_depth_py" value="0.0175"/>
+    <xacro:property name="d435i_cam_depth_pz" value="${d435i_cam_height/2}"/>
+    <material name="${name}_aluminum">
+	  <color rgba="0.5 0.5 0.5 1"/>
+    </material>
+    <!-- camera body, with origin at bottom screw mount -->
+    <joint name="${name}_joint" type="fixed">
+      <xacro:insert_block name="origin"/>
+      <parent link="${parent}"/>
+      <child link="${name}_bottom_screw_frame"/>
+    </joint>
+    <link name="${name}_bottom_screw_frame"/>
+    <joint name="${name}_link_joint" type="fixed">
+      <origin xyz="0 ${d435i_cam_depth_py} ${d435i_cam_depth_pz}" rpy="0 0 0"/>
+      <parent link="${name}_bottom_screw_frame"/>
+      <child link="${name}_link"/>
+    </joint>
+    <link name="${name}_link">
+      <visual>
+      <origin xyz="${d435i_cam_mount_from_center_offset} ${-d435i_cam_depth_py} 0" rpy="${M_PI/2} 0 ${M_PI/2}"/>
+        <geometry>
+          <mesh filename="../../meshes/d435.dae"/>
+        </geometry>
+        <material name="${name}_aluminum"/>
+      </visual>
+      <collision>
+        <origin xyz="0 ${-d435i_cam_depth_py} 0" rpy="0 0 0"/>
+        <geometry>
+        <box size="${d435i_cam_depth} ${d435i_cam_width} ${d435i_cam_height}"/>
+        </geometry>
+      </collision>
+      <inertial>
+        <!-- The following are not reliable values, and should not be used for modeling -->
+        <mass value="0.564"/>
+        <origin xyz="0 0 0"/>
+        <inertia ixx="0.003881243" ixy="0.0" ixz="0.0" iyy="0.000498940" iyz="0.0" izz="0.003879257"/>
+      </inertial>
+    </link>
+    <!-- camera depth joints and links -->
+    <joint name="${name}_depth_joint" type="fixed">
+      <origin xyz="0 0 0" rpy="0 0 0"/>
+      <parent link="${name}_link"/>
+      <child link="${name}_depth_frame"/>
+    </joint>
+    <link name="${name}_depth_frame"/>
+    <joint name="${name}_depth_optical_joint" type="fixed">
+      <origin xyz="0 0 0" rpy="${-M_PI/2} 0 ${-M_PI/2}"/>
+      <parent link="${name}_depth_frame"/>
+      <child link="${name}_depth_optical_frame"/>
+    </joint>
+    <link name="${name}_depth_optical_frame"/>
+    <!-- camera left IR joints and links -->
+    <joint name="${name}_left_ir_joint" type="fixed">
+      <origin xyz="0 ${d435i_cam_depth_to_left_ir_offset} 0" rpy="0 0 0"/>
+      <parent link="${name}_depth_frame"/>
+      <child link="${name}_left_ir_frame"/>
+    </joint>
+    <link name="${name}_left_ir_frame"/>
+    <joint name="${name}_left_ir_optical_joint" type="fixed">
+      <origin xyz="0 0 0" rpy="${-M_PI/2} 0 ${-M_PI/2}"/>
+      <parent link="${name}_left_ir_frame"/>
+      <child link="${name}_left_ir_optical_frame"/>
+    </joint>
+    <link name="${name}_left_ir_optical_frame"/>
+    <!-- camera right IR joints and links -->
+    <joint name="${name}_right_ir_joint" type="fixed">
+      <origin xyz="0 ${d435i_cam_depth_to_right_ir_offset} 0" rpy="0 0 0"/>
+      <parent link="${name}_depth_frame"/>
+      <child link="${name}_right_ir_frame"/>
+    </joint>
+    <link name="${name}_right_ir_frame"/>
+    <joint name="${name}_right_ir_optical_joint" type="fixed">
+      <origin xyz="0 0 0" rpy="${-M_PI/2} 0 ${-M_PI/2}"/>
+      <parent link="${name}_right_ir_frame"/>
+      <child link="${name}_right_ir_optical_frame"/>
+    </joint>
+    <link name="${name}_right_ir_optical_frame"/>
+    <!-- camera color joints and links -->
+    <joint name="${name}_color_joint" type="fixed">
+      <origin xyz="0 ${d435i_cam_depth_to_color_offset} 0" rpy="0 0 0"/>
+      <parent link="${name}_depth_frame"/>
+      <child link="${name}_color_frame"/>
+    </joint>
+    <link name="${name}_color_frame"/>
+    <joint name="${name}_color_optical_joint" type="fixed">
+      <origin xyz="0 0 0" rpy="${-M_PI/2} 0 ${-M_PI/2}"/>
+      <parent link="${name}_color_frame"/>
+      <child link="${name}_color_optical_frame"/>
+    </joint>
+    <link name="${name}_color_optical_frame"/>
+    <!-- camera accel joints and links -->
+    <joint name="${name}_accel_joint" type="fixed">
+      <origin xyz="-0.00174 0.00552 0.0176" rpy="0 0 0"/>
+      <parent link="${name}_link"/>
+      <child link="${name}_accel_frame"/>
+    </joint>
+    <link name="${name}_accel_frame"/>
+    <joint name="${name}_accel_optical_joint" type="fixed">
+      <origin xyz="0 0 0" rpy="${-M_PI/2} 0 ${-M_PI/2}"/>
+      <parent link="${name}_accel_frame"/>
+      <child link="${name}_accel_optical_frame"/>
+    </joint>
+    <link name="${name}_accel_optical_frame"/>
+    <!-- camera gyro joints and links -->
+    <joint name="${name}_gyro_joint" type="fixed">
+      <origin xyz="-0.00174 0.00552 0.0176" rpy="0 0 0"/>
+      <parent link="${name}_link"/>
+      <child link="${name}_gyro_frame"/>
+    </joint>
+    <link name="${name}_gyro_frame"/>
+    <joint name="${name}_gyro_optical_joint" type="fixed">
+      <origin xyz="0 0 0" rpy="${-M_PI/2} 0 ${-M_PI/2}"/>
+      <parent link="${name}_gyro_frame"/>
+      <child link="${name}_gyro_optical_frame"/>
+    </joint>
+    <link name="${name}_gyro_optical_frame"/>
+    <!-- Realsense Gazebo Plugin -->
+    <xacro:gazebo_d435i camera_name="${name}"
+                        topics_ns="${topics_ns}"
+                        reference_link="${name}_link"
+                        depth_optical_frame="${name}_depth_optical_frame"
+                        depth_width="${depth_width}"
+                        depth_height="${depth_height}"
+                        depth_fps="${depth_fps}"
+                        color_optical_frame="${name}_color_optical_frame"
+                        color_width="${color_width}"
+                        color_height="${color_height}"
+                        color_fps="${color_fps}"
+                        infrared1_optical_frame="${name}_left_ir_optical_frame"
+                        infrared2_optical_frame="${name}_right_ir_optical_frame"
+                        infra_width="${infra_width}"
+                        infra_height="${infra_height}"
+                        infra_fps="${infra_fps}"
+                        accel_optical_frame="${name}_accel_optical_frame"
+                        gyro_optical_frame="${name}_gyro_optical_frame"
+                        accel_fps="${accel_fps}"
+                        gyro_fps="${gyro_fps}"
+                        enable_pointCloud="${enable_pointCloud}"
+                        unite_imu_method="${unite_imu_method}"
+                        clip_distance="${clip_distance}"
+                        align_depth="${align_depth}"
+                        visualize="${visualize}"
+    />
+  </xacro:macro>
+   <xacro:macro name="gazebo_d435i" params=" reference_link
+                                            camera_name:=camera
+                                            topics_ns:=camera
+                                            depth_optical_frame
+                                            color_optical_frame
+                                            infrared1_optical_frame
+                                            infrared2_optical_frame
+                                            accel_optical_frame
+                                            gyro_optical_frame
+                                            visualize:=false
+                                            align_depth:=false
+                                            enable_pointCloud:=false
+                                            unite_imu_method:=false
+                                            accel_fps:=250
+                                            gyro_fps:=400
+                                            clip_distance:=-1.0
+                                            depth_width:=1280
+                                            depth_height:=720
+                                            depth_fps:=30
+                                            infra_width:=640
+                                            infra_height:=480
+                                            infra_fps:=30
+                                            color_width:=1920
+                                            color_height:=1080
+                                            color_fps:=30
+                                            ">
+    <!-- Load parameters to model's main link-->
+    <xacro:property name="deg_to_rad" value="0.01745329251994329577"/>
+    <gazebo reference="${reference_link}">
+      <self_collide>0</self_collide>
+      <enable_wind>0</enable_wind>
+      <kinematic>0</kinematic>
+      <!-- <gravity>1</gravity> -->
+      <!--<mu>1</mu>-->
+      <mu2>1</mu2>
+      <fdir1>0 0 0</fdir1>
+      <!--<slip1>0</slip1>
+      <slip2>0</slip2>-->
+      <kp>1e+13</kp>
+      <kd>1</kd>
+      <!--<max_vel>0.01</max_vel>
+      <min_depth>0</min_depth>-->
+      <sensor name="${camera_name}color" type="camera">
+        <camera name="${camera_name}">
+          <horizontal_fov>${69.4*deg_to_rad}</horizontal_fov>
+          <image>
+            <width>${color_width}</width>
+            <height>${color_height}</height>
+            <format>RGB_INT8</format>
+          </image>
+          <clip>
+            <near>0.1</near>
+            <far>100</far>
+          </clip>
+          <noise>
+            <type>gaussian</type>
+            <mean>0.0</mean>
+            <stddev>0.007</stddev>
+          </noise>
+        </camera>
+        <always_on>1</always_on>
+        <update_rate>${color_fps}</update_rate>
+        <visualize>${visualize}</visualize>
+      </sensor>
+      <sensor name="${camera_name}ired1" type="camera">
+        <camera name="${camera_name}">
+          <horizontal_fov>${85.2*deg_to_rad}</horizontal_fov>
+          <image>
+            <width>${infra_width}</width>
+            <height>${infra_height}</height>
+            <format>L_INT8</format>
+          </image>
+          <clip>
+            <near>0.1</near>
+            <far>100</far>
+          </clip>
+          <noise>
+            <type>gaussian</type>
+            <mean>0.0</mean>
+            <stddev>0.05</stddev>
+          </noise>
+        </camera>
+        <always_on>1</always_on>
+        <update_rate>${infra_fps}</update_rate>
+        <visualize>false</visualize>
+      </sensor>
+      <sensor name="${camera_name}ired2" type="camera">
+        <camera name="${camera_name}">
+          <horizontal_fov>${85.2*deg_to_rad}</horizontal_fov>
+          <image>
+            <width>${infra_width}</width>
+            <height>${infra_height}</height>
+            <format>L_INT8</format>
+          </image>
+          <clip>
+            <near>0.1</near>
+            <far>100</far>
+          </clip>
+          <noise>
+            <type>gaussian</type>
+            <mean>0.0</mean>
+            <stddev>0.05</stddev>
+          </noise>
+        </camera>
+        <always_on>1</always_on>
+        <update_rate>${infra_fps}</update_rate>
+        <visualize>false</visualize>
+      </sensor>
+      <sensor name="${camera_name}depth" type="depth">
+        <camera name="${camera_name}">
+          <!-- align-depth settings -->
+          <xacro:unless value="${align_depth}">
+            <horizontal_fov>${85.2*deg_to_rad}</horizontal_fov>
+            <image>
+              <width>${depth_width}</width>
+              <height>${depth_height}</height>
+            </image>
+          </xacro:unless>
+          <xacro:if value="${align_depth}">
+            <horizontal_fov>${69.4*deg_to_rad}</horizontal_fov>
+            <image>
+              <width>${color_width}</width>
+              <height>${color_height}</height>
+            </image>
+          </xacro:if>
+          <clip>
+            <near>0.1</near>
+            <xacro:unless value="${clip_distance > 0.0}">
+              <far>100</far>
+            </xacro:unless>
+            <xacro:if value="${clip_distance > 0.0}">
+              <far>${clip_distance}</far>
+            </xacro:if>
+          </clip>
+          <noise>
+            <type>gaussian</type>
+            <mean>0.0</mean>
+            <stddev>0.100</stddev>
+          </noise>
+        </camera>
+        <always_on>1</always_on>
+        <xacro:unless value="${align_depth}">
+          <update_rate>${depth_fps}</update_rate>
+        </xacro:unless>
+        <xacro:if value="${align_depth}">
+          <update_rate>${color_fps}</update_rate>
+        </xacro:if>
+        <visualize>false</visualize>
+      </sensor>
+      <!-- IMU -->
+      <xacro:if value="${unite_imu_method == 'copy' or unite_imu_method == 'linear_interpolation'}">
+        <sensor name="${camera_name}imu" type="imu">
+          <always_on>true</always_on>
+          <update_rate>${gyro_fps}</update_rate>
+          <topic>${camera_name}/imu/sample</topic>
+          <plugin name="${camera_name}imu" filename="libgazebo_ros_imu_sensor.so">
+            <topicName>${camera_name}/imu/sample</topicName>
+            <bodyName>${camera_name}_link</bodyName>
+            <frameName>${gyro_optical_frame}</frameName>
+            <updateRateHZ>${gyro_fps}</updateRateHZ>
+            <gaussianNoise>0.1</gaussianNoise>
+            <xyzOffset>0 0 0</xyzOffset>
+            <rpyOffset>0 0 0</rpyOffset>
+          </plugin>
+        </sensor>
+      </xacro:if>
+      <!-- Accel and gyro -->
+      <xacro:unless value="${unite_imu_method == 'copy' or unite_imu_method == 'linear_interpolation'}">
+        <sensor name="${camera_name}accel" type="imu">
+          <always_on>true</always_on>
+          <update_rate>${accel_fps}</update_rate>
+          <topic>${camera_name}/accel/sample</topic>
+          <plugin name="${topics_ns}_accel_plugin" filename="librealsense_gazebo_accel_sensor.so">
+            <topicName>${camera_name}/accel/sample</topicName>
+            <bodyName>${camera_name}_link</bodyName>
+            <updateRateHZ>${accel_fps}</updateRateHZ>
+            <gaussianNoise>0.1</gaussianNoise>
+            <xyzOffset>0 0 0</xyzOffset>
+            <rpyOffset>0 0 0</rpyOffset>
+            <frameName>${accel_optical_frame}</frameName>
+            <initialOrientationAsReference>false</initialOrientationAsReference>
+          </plugin>
+          <pose>0 0 0 0 0 0</pose>
+        </sensor>
+        <sensor name="${camera_name}gyro" type="imu">
+          <always_on>true</always_on>
+          <update_rate>${gyro_fps}</update_rate>
+          <topic>${camera_name}/gyro/sample</topic>
+          <plugin name="${topics_ns}_gyro_plugin" filename="librealsense_gazebo_gyro_sensor.so">
+            <topicName>${camera_name}/gyro/sample</topicName>
+            <bodyName>${camera_name}_link</bodyName>
+            <updateRateHZ>${gyro_fps}</updateRateHZ>
+            <gaussianNoise>0.1</gaussianNoise>
+            <xyzOffset>0 0 0</xyzOffset>
+            <rpyOffset>0 0 0</rpyOffset>
+            <frameName>${gyro_optical_frame}</frameName>
+            <initialOrientationAsReference>false</initialOrientationAsReference>
+          </plugin>
+        </sensor>
+      </xacro:unless>
+    </gazebo>
+    <gazebo>
+      <plugin name="${topics_ns}" filename="librealsense_gazebo_plugin.so">
+        <prefix>${camera_name}</prefix>
+        <!-- Color camera settings -->
+      	<colorUpdateRate>${color_fps}</colorUpdateRate>
+      	<colorTopicName>color/image_raw</colorTopicName>
+      	<colorOpticalframeName>${color_optical_frame}</colorOpticalframeName>
+      	<colorCameraInfoTopicName>color/camera_info</colorCameraInfoTopicName>
+        <!-- Infrared camera settings -->
+      	<infraredUpdateRate>${infra_fps}</infraredUpdateRate>
+      	<infrared1TopicName>infra1/image_rect_raw</infrared1TopicName>
+      	<infrared2TopicName>infra2/image_rect_raw</infrared2TopicName>
+      	<infrared1CameraInfoTopicName>infra1/camera_info</infrared1CameraInfoTopicName>
+      	<infrared2CameraInfoTopicName>infra2/camera_info</infrared2CameraInfoTopicName>
+      	<infrared1OpticalframeName>${infrared1_optical_frame}</infrared1OpticalframeName>
+      	<infrared2OpticalframeName>${infrared2_optical_frame}</infrared2OpticalframeName>
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