Commit message: optimized moveit config

File: src/meca500_moveit_config/config/meca500.ros2_control.xacro (robot description, xacro)
@@ -9,44 +9,14 @@
             </hardware>
             <joint name="meca_axis_1_joint">
-                <command_interface name="velocity"/>
-                <state_interface name="position">
-                  <param name="initial_value">${initial_positions['meca_axis_1_joint']}</param>
-                </state_interface>
-                <state_interface name="velocity"/>
             </joint>
             <joint name="meca_axis_2_joint">
-                <command_interface name="velocity"/>
-                <state_interface name="position">
-                  <param name="initial_value">${initial_positions['meca_axis_2_joint']}</param>
-                </state_interface>
-                <state_interface name="velocity"/>
             </joint>
             <joint name="meca_axis_3_joint">
-                <command_interface name="velocity"/>
-                <state_interface name="position">
-                  <param name="initial_value">${initial_positions['meca_axis_3_joint']}</param>
-                </state_interface>
-                <state_interface name="velocity"/>
             </joint>
             <joint name="meca_axis_4_joint">
-                <command_interface name="velocity"/>
-                <state_interface name="position">
-                  <param name="initial_value">${initial_positions['meca_axis_4_joint']}</param>
-                </state_interface>
-                <state_interface name="velocity"/>
             </joint>
             <joint name="meca_axis_5_joint">
-                <command_interface name="velocity"/>
-                <state_interface name="position">
-                  <param name="initial_value">${initial_positions['meca_axis_5_joint']}</param>
-                </state_interface>
-                <state_interface name="velocity"/>
             </joint>
             <joint name="meca_axis_6_joint">
-                <command_interface name="velocity"/>
-                <state_interface name="position">
-                  <param name="initial_value">${initial_positions['meca_axis_6_joint']}</param>
-                </state_interface>
-                <state_interface name="velocity"/>
             </joint>
         </ros2_control>

File: src/meca500_moveit_config/config/meca500.urdf.xacro (robot description, xacro)
@@ -3,5 +3,5 @@
     <xacro:arg name="initial_positions_file" default="initial_positions.yaml" />
     <!-- Import meca500 urdf file -->
-    <xacro:include filename="$(find meca500_world)/models/meca500/meca500_pkg_reference.xacro" />
+    <xacro:include filename="$(find meca500_world)/models/meca500/meca500.xacro" />
     <!-- Import control_xacro -->
     <xacro:include filename="meca500.ros2_control.xacro" />

File: src/meca500_world/models/meca500/meca500.xacro (robot description, xacro)
@@ -32,9 +32,4 @@
                                           *origin">
     <xacro:property name="M_PI" value="3.1415926535897931"/>
-    <!-- The following values are approximate, and the camera node
-     publishing TF values with actual calibrated camera extrinsic values -->
-    <xacro:property name="d435i_cam_depth_to_left_ir_offset" value="0.0"/>
-    <xacro:property name="d435i_cam_depth_to_right_ir_offset" value="-0.050"/>
-    <xacro:property name="d435i_cam_depth_to_color_offset" value="0.015"/>
     <!-- The following values model the aluminum peripherial case for the
   	D435 camera, with the camera joint represented by the actual
@@ -85,82 +80,4 @@
       </inertial>
     </link>
-    <!-- camera depth joints and links -->
-    <joint name="${name}_depth_joint" type="fixed">
-      <origin xyz="0 0 0" rpy="0 0 0"/>
-      <parent link="${name}_link"/>
-      <child link="${name}_depth_frame"/>
-    </joint>
-    <link name="${name}_depth_frame"/>
-    <joint name="${name}_depth_optical_joint" type="fixed">
-      <origin xyz="0 0 0" rpy="${-M_PI/2} 0 ${-M_PI/2}"/>
-      <parent link="${name}_depth_frame"/>
-      <child link="${name}_depth_optical_frame"/>
-    </joint>
-    <link name="${name}_depth_optical_frame"/>
-    <!-- camera left IR joints and links -->
-    <joint name="${name}_left_ir_joint" type="fixed">
-      <origin xyz="0 ${d435i_cam_depth_to_left_ir_offset} 0" rpy="0 0 0"/>
-      <parent link="${name}_depth_frame"/>
-      <child link="${name}_left_ir_frame"/>
-    </joint>
-    <link name="${name}_left_ir_frame"/>
-    <joint name="${name}_left_ir_optical_joint" type="fixed">
-      <origin xyz="0 0 0" rpy="${-M_PI/2} 0 ${-M_PI/2}"/>
-      <parent link="${name}_left_ir_frame"/>
-      <child link="${name}_left_ir_optical_frame"/>
-    </joint>
-    <link name="${name}_left_ir_optical_frame"/>
-    <!-- camera right IR joints and links -->
-    <joint name="${name}_right_ir_joint" type="fixed">
-      <origin xyz="0 ${d435i_cam_depth_to_right_ir_offset} 0" rpy="0 0 0"/>
-      <parent link="${name}_depth_frame"/>
-      <child link="${name}_right_ir_frame"/>
-    </joint>
-    <link name="${name}_right_ir_frame"/>
-    <joint name="${name}_right_ir_optical_joint" type="fixed">
-      <origin xyz="0 0 0" rpy="${-M_PI/2} 0 ${-M_PI/2}"/>
-      <parent link="${name}_right_ir_frame"/>
-      <child link="${name}_right_ir_optical_frame"/>
-    </joint>
-    <link name="${name}_right_ir_optical_frame"/>
-    <!-- camera color joints and links -->
-    <joint name="${name}_color_joint" type="fixed">
-      <origin xyz="0 ${d435i_cam_depth_to_color_offset} 0" rpy="0 0 0"/>
-      <parent link="${name}_depth_frame"/>
-      <child link="${name}_color_frame"/>
-    </joint>
-    <link name="${name}_color_frame"/>
-    <joint name="${name}_color_optical_joint" type="fixed">
-      <origin xyz="0 0 0" rpy="${-M_PI/2} 0 ${-M_PI/2}"/>
-      <parent link="${name}_color_frame"/>
-      <child link="${name}_color_optical_frame"/>
-    </joint>
-    <link name="${name}_color_optical_frame"/>
-    <!-- camera accel joints and links -->
-    <joint name="${name}_accel_joint" type="fixed">
-      <origin xyz="-0.00174 0.00552 0.0176" rpy="0 0 0"/>
-      <parent link="${name}_link"/>
-      <child link="${name}_accel_frame"/>
-    </joint>
-    <link name="${name}_accel_frame"/>
-    <joint name="${name}_accel_optical_joint" type="fixed">
-      <origin xyz="0 0 0" rpy="${-M_PI/2} 0 ${-M_PI/2}"/>
-      <parent link="${name}_accel_frame"/>
-      <child link="${name}_accel_optical_frame"/>
-    </joint>
-    <link name="${name}_accel_optical_frame"/>
-    <!-- camera gyro joints and links -->
-    <joint name="${name}_gyro_joint" type="fixed">
-      <origin xyz="-0.00174 0.00552 0.0176" rpy="0 0 0"/>
-      <parent link="${name}_link"/>
-      <child link="${name}_gyro_frame"/>
-    </joint>
-    <link name="${name}_gyro_frame"/>
-    <joint name="${name}_gyro_optical_joint" type="fixed">
-      <origin xyz="0 0 0" rpy="${-M_PI/2} 0 ${-M_PI/2}"/>
-      <parent link="${name}_gyro_frame"/>
-      <child link="${name}_gyro_optical_frame"/>
-    </joint>
-    <link name="${name}_gyro_optical_frame"/>
     <!-- Realsense Gazebo Plugin -->
     <xacro:gazebo_d435i camera_name="${name}"
